File: VFD Clock.kicad_sch (KiCad schematic)
At the start: 4 parts, among them U1 74HC595, U2 UDN2981A, U3 IV-11 VFD Tube

Commit message: saving
Parts:
- added U10, U13, U16, U4, U7: 74HC595, Package_DIP:DIP-16_W7.62mm, symbol 74xx:74HC595
- added U11, U14, U17, U5, U8: UDN2981A, UDN2981A:DIP254P762X533-18, symbol UDN2981A:UDN2981A
- added U12, U15, U18, U6, U9: IV-11 VFD Tube, Custom Parts:IV-11 VFD Tube, symbol Custom Parts:IV-11_VFD_Tube
Connections:
- net +1.5V: now also U12.11 (Fil), U15.11 (Fil), U18.11 (Fil), U6.11 (Fil), U9.11 (Fil)
- net +25V: now also U3.2 (Grid), U11.9 (VS), U12.2 (Grid), U14.9 (VS), U15.2 (Grid), U17.9 (VS), U18.2 (Grid), U5.9 (VS), U6.2 (Grid), U8.9 (VS), U9.2 (Grid)
- net +5V: now also U1.10 (~{SRCLR}), U10.10 (~{SRCLR}), U10.16 (VCC), U13.10 (~{SRCLR}), U13.16 (VCC), U16.10 (~{SRCLR}), U16.16 (VCC), U4.10 (~{SRCLR}), U4.16 (VCC), U7.10 (~{SRCLR}), U7.16 (VCC)
- net GND: now also U1.13 (~{OE}), U10.13 (~{OE}), U10.8 (GND), U11.10 (GND), U12.1 (Fil), U13.13 (~{OE}), U13.8 (GND), U14.10 (GND), U15.1 (Fil), U16.13 (~{OE}), U16.8 (GND), U17.10 (GND), U18.1 (Fil), U4.13 (~{OE}), U4.8 (GND), U5.10 (GND), U6.1 (Fil), U7.13 (~{OE}), U7.8 (GND), U8.10 (GND), U9.1 (Fil)
- net Latch: now reaches A1.14 (MOSI)
- net Latch: now also U1.12 (RCLK), U10.12 (RCLK), U13.12 (RCLK), U16.12 (RCLK), U4.12 (RCLK), U7.12 (RCLK)
- net Data: now reaches A1.15 (MISO)
- net Data: now also U1.14 (SER)
- net Shift: now reaches A1.16 (SCK)
- net Shift: now also U1.11 (SRCLK), U10.11 (SRCLK), U13.11 (SRCLK), U16.11 (SRCLK), U4.11 (SRCLK), U7.11 (SRCLK)
- net SDA: now reaches A1.23 (SDA/A4)
- net SCL: now reaches A1.24 (SCL/A5)
- net at U1.9 (QH'): now also U4.14 (SER)
- new net: U7.15 (QA), U8.1 (IN1)
- new net: U8.11 (OUT8), U9.10 (H)
- new net: U8.12 (OUT7), U9.9 (G)
- new net: U8.13 (OUT6), U9.8 (F)
- new net: U8.14 (OUT5), U9.7 (E)
- new net: U8.15 (OUT4), U9.6 (D)
- new net: U8.16 (OUT3), U9.5 (C)
- new net: U8.17 (OUT2), U9.4 (B)
- new net: U8.18 (OUT1), U9.3 (A)
- new net: U7.1 (QB), U8.2 (IN2)
- new net: U7.2 (QC), U8.3 (IN3)
- new net: U7.3 (QD), U8.4 (IN4)
- new net: U7.4 (QE), U8.5 (IN5)
- new net: U7.5 (QF), U8.6 (IN6)
- new net: U7.6 (QG), U8.7 (IN7)
- new net: U7.7 (QH), U8.8 (IN8)
- new net: U11.11 (OUT8), U12.10 (H)
- new net: U11.18 (OUT1), U12.3 (A)
- new net: U11.17 (OUT2), U12.4 (B)
- new net: U11.16 (OUT3), U12.5 (C)
- new net: U11.15 (OUT4), U12.6 (D)
- new net: U11.14 (OUT5), U12.7 (E)
- new net: U11.13 (OUT6), U12.8 (F)
- new net: U11.12 (OUT7), U12.9 (G)
- new net: U10.15 (QA), U11.1 (IN1)
- new net: U10.1 (QB), U11.2 (IN2)
- new net: U10.2 (QC), U11.3 (IN3)
- new net: U10.3 (QD), U11.4 (IN4)
- new net: U10.4 (QE), U11.5 (IN5)
- new net: U10.5 (QF), U11.6 (IN6)
- new net: U10.6 (QG), U11.7 (IN7)
- new net: U10.7 (QH), U11.8 (IN8)
- new net: U13.1 (QB), U14.2 (IN2)
- new net: U10.9 (QH'), U13.14 (SER)
- new net: U13.15 (QA), U14.1 (IN1)
- new net: U13.2 (QC), U14.3 (IN3)
- new net: U13.3 (QD), U14.4 (IN4)
- new net: U13.4 (QE), U14.5 (IN5)
- new net: U13.5 (QF), U14.6 (IN6)
- new net: U13.6 (QG), U14.7 (IN7)
- new net: U13.7 (QH), U14.8 (IN8)
- new net: U13.9 (QH'), U16.14 (SER)
- new net: U5.11 (OUT8), U6.10 (H)
- new net: U5.18 (OUT1), U6.3 (A)
- new net: U5.17 (OUT2), U6.4 (B)
- new net: U5.16 (OUT3), U6.5 (C)
- new net: U5.15 (OUT4), U6.6 (D)
- new net: U5.14 (OUT5), U6.7 (E)
- new net: U5.13 (OUT6), U6.8 (F)
- new net: U5.12 (OUT7), U6.9 (G)
- new net: U16.15 (QA), U17.1 (IN1)
- new net: U17.11 (OUT8), U18.10 (H)
- new net: U17.12 (OUT7), U18.9 (G)
- new net: U17.13 (OUT6), U18.8 (F)
- new net: U17.14 (OUT5), U18.7 (E)
- new net: U17.15 (OUT4), U18.6 (D)
- new net: U17.16 (OUT3), U18.5 (C)
- new net: U17.17 (OUT2), U18.4 (B)
- new net: U17.18 (OUT1), U18.3 (A)
- new net: U16.1 (QB), U17.2 (IN2)
- new net: U16.2 (QC), U17.3 (IN3)
- new net: U16.3 (QD), U17.4 (IN4)
- new net: U16.4 (QE), U17.5 (IN5)
- new net: U16.5 (QF), U17.6 (IN6)
- new net: U16.6 (QG), U17.7 (IN7)
- new net: U16.7 (QH), U17.8 (IN8)
- new net: U14.11 (OUT8), U15.10 (H)
- new net: U14.18 (OUT1), U15.3 (A)
- new net: U14.17 (OUT2), U15.4 (B)
- new net: U14.16 (OUT3), U15.5 (C)
- new net: U14.15 (OUT4), U15.6 (D)
- new net: U14.14 (OUT5), U15.7 (E)
- new net: U14.13 (OUT6), U15.8 (F)
- new net: U14.12 (OUT7), U15.9 (G)
- new net: U4.15 (QA), U5.1 (IN1)
- new net: U4.1 (QB), U5.2 (IN2)
- new net: U4.2 (QC), U5.3 (IN3)
- new net: U4.3 (QD), U5.4 (IN4)
- new net: U4.4 (QE), U5.5 (IN5)
- new net: U4.5 (QF), U5.6 (IN6)
- new net: U4.6 (QG), U5.7 (IN7)
- new net: U4.7 (QH), U5.8 (IN8)
- new net: U4.9 (QH'), U7.14 (SER)
- new net: U10.14 (SER), U7.9 (QH')
Other:
- moved on the sheet: A1, U1, U2, U3

Commit message: saving
Parts:
- added C1: 100uF, Capacitor_THT:CP_Radial_D6.3mm_P2.50mm, symbol Device:C
- added C2, C3, C4, C5, C6, C7: 100nF, Capacitor_THT:CP_Radial_D6.3mm_P2.50mm, symbol Device:C
- added J1: DS3231, symbol Connector:Conn_01x04_Socket
Connections:
- net +5V: now also C1.1, C2.1, C3.1, C4.1, C5.1, C6.1, C7.1, J1.3 (Pin_3)
- net GND: now also C1.2, C2.2, C3.2, C4.2, C5.2, C6.2, C7.2, J1.4 (Pin_4)
- net SCL: now also J1.1 (Pin_1)
- net SDA: now also J1.2 (Pin_2)
- no-connect marks 0 -> 1
Other:
- moved on the sheet: A1
