File: VFD Clock.kicad_pcb (KiCad board)
At the start: 2 copper layers, 220 x 78.5 mm, 37 parts, among them J2 Mode Button, J3 Up Button, J4 Down Button, J5 Select Button, U1 74HC595, U10 74HC595, U11 UDN2981A, U12 Minute Right, U13 74HC595, U14 UDN2981A, U15 Second Left, U16 74HC595, U17 UDN2981A, U18 Second Right, U19 XL6009 Module, U2 UDN2981A, U20 LM2596 Module, U21 DS3231 Module, U3 Hour Left, U4 74HC595, U5 UDN2981A, U6 Hour Right, U7 74HC595, U8 UDN2981A, U9 Minute Left

Commit message: save
Parts:
- moved C10 24.5 mm to (112.5, 119.0)
- moved REF** 2.12 mm to (66.9, 75.0)
- moved REF** 2.06 mm to (66.9, 146.5)
- moved REF** 2.00 mm to (284.0, 146.5)
- moved REF** 2.00 mm to (284.0, 75.0)
Other:
- board size 220 x 78.5 mm -> 224 x 78.5 mm
Changed lines of the file:
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@@
 	(footprint "MountingHole:MountingHole_3.2mm_M3"
 		(layer "F.Cu")
-		(at 69 75)
+		(at 66.881135 74.954983)
 		(descr "Mounting Hole 3.2mm, M3, no annular, generated by kicad-footprint-generator mountinghole.py")
 		(tags "mountinghole M3")
@@
 	(footprint "MountingHole:MountingHole_3.2mm_M3"
 		(layer "F.Cu")
-		(at 282 146.5)
+		(at 284 146.5)
 		(descr "Mounting Hole 3.2mm, M3, no annular, generated by kicad-footprint-generator mountinghole.py")
 		(tags "mountinghole M3")
@@
 	(footprint "MountingHole:MountingHole_3.2mm_M3"
 		(layer "F.Cu")
-		(at 69 146.5)
+		(at 66.945211 146.450088)
 		(descr "Mounting Hole 3.2mm, M3, no annular, generated by kicad-footprint-generator mountinghole.py")
 		(tags "mountinghole M3")
@@
 	(footprint "MountingHole:MountingHole_3.2mm_M3"
 		(layer "F.Cu")
-		(at 282 75)
+		(at 284 75)
 		(descr "Mounting Hole 3.2mm, M3, no annular, generated by kicad-footprint-generator mountinghole.py")
 		(tags "mountinghole M3")
@@
 			(at 22 -10.5 0)
 			(unlocked yes)
-			(layer "B.Fab")
+			(layer "B.SilkS")
 			(effects
 				(font
@@
 		(property "Value" "UDN2981A"
 			(at -10 4.16 0)
-			(layer "B.Fab")
+			(layer "B.SilkS")
 			(effects
 				(font
@@
 		)
 		(property "Value" "74HC595"
-			(at -1.997706 -19.497842 0)
-			(layer "B.Fab")
+			(at 10 -16 0)
+			(layer "B.SilkS")
 			(effects
 				(font
@@
 		)
 		(property "Value" "74HC595"
-			(at -2.192706 -21.577842 0)
-			(layer "B.Fab")
+			(at 9.807294 -16 0)
+			(layer "B.SilkS")
 			(effects
 				(font
@@
 			(at 1.25 4.4 0)
 			(layer "B.SilkS")
+			(hide yes)
 			(effects
 				(font
@@
 		(property "Value" "100uF"
 			(at 1.25 -4.4 0)
-			(layer "B.Fab")
+			(layer "B.SilkS")
 			(effects
 				(font
@@
 		)
 		(property "Value" "74HC595"
-			(at -1.997706 -14.497842 0)
-			(layer "B.Fab")
+			(at 10 -16 0)
+			(layer "B.SilkS")
 			(effects
 				(font
@@
 		)
 		(property "Value" "74HC595"
-			(at -2.192706 -18.387842 0)
-			(layer "B.Fab")
+			(at 10 -16 0)
+			(layer "B.SilkS")
 			(effects
 				(font
@@
 		(property "Value" "Mode Button"
 			(at -3 -1.5 0)
-			(layer "B.Fab")
+			(layer "B.SilkS")
 			(effects
 				(font
@@
 		)
 		(property "Value" "Select Button"
-			(at -3 -2.5 0)
-			(layer "B.Fab")
+			(at -3 -1 0)
+			(layer "B.SilkS")
 			(effects
 				(font
@@
 		)
 		(property "Value" "100nF"
-			(at 0.997706 3.497842 0)
-			(layer "B.Fab")
+			(at -2.002294 -0.497842 0)
+			(layer "B.SilkS")
 			(effects
 				(font
@@
 		(property "Value" "UDN2981A"
 			(at -10 5 0)
-			(layer "B.Fab")
+			(layer "B.SilkS")
 			(effects
 				(font
@@
 		)
 		(property "Value" "Down Button"
-			(at -3 -2 0)
-			(layer "B.Fab")
+			(at -3 -1 0)
+			(layer "B.SilkS")
 			(effects
 				(font
@@
 			(at 25.4 -10.16 0)
 			(unlocked yes)
-			(layer "B.Fab")
+			(layer "B.SilkS")
 			(effects
 				(font
@@
 			(at 7.62 5.08 0)
 			(layer "B.SilkS")
+			(hide yes)
 			(effects
 				(font
@@
 		(property "Value" "Arduino_Nano_Every"
 			(at 8.89 -19.05 90)
-			(layer "B.Fab")
+			(layer "B.SilkS")
 			(effects
 				(font
@@
 		)
 		(property "Value" "100nF"
-			(at 1.25 -2.05 90)
-			(layer "B.Fab")
+			(at -2.002294 -1.497842 0)
+			(layer "B.SilkS")
 			(effects
 				(font
@@
 		)
 		(property "Value" "100nF"
-			(at 0.997706 3.497842 0)
-			(layer "B.Fab")
+			(at -2.002294 -0.497842 0)
+			(layer "B.SilkS")
 			(effects
 				(font
@@
 		)
 		(property "Value" "UDN2981A"
-			(at -10 4.696 0)
-			(layer "B.Fab")
+			(at -10.001344 4.680885 0)
+			(layer "B.SilkS")
 			(effects
 				(font
@@
 		)
 		(property "Value" "UDN2981A"
-			(at -10 3.928 0)
-			(layer "B.Fab")
+			(at -10.001344 4.920683 0)
+			(layer "B.SilkS")
 			(effects
 				(font
@@
 		(property "Value" "UDN2981A"
 			(at -10 5.464 0)
-			(layer "B.Fab")
+			(layer "B.SilkS")
 			(effects
 				(font
@@
 		)
 		(property "Value" "100nF"
-			(at 0.997706 3.497842 0)
-			(layer "B.Fab")
+			(at -2.002294 -0.497842 0)
+			(layer "B.SilkS")
 			(effects
 				(font
@@
 			(at 21 -7.5 0)
 			(unlocked yes)
-			(layer "B.Fab")
+			(layer "B.SilkS")
 			(effects
 				(font
@@
 		)
 		(property "Value" "74HC595"
-			(at -1.997706 -18.497842 0)
-			(layer "B.Fab")
+			(at 10 -16 0)
+			(layer "B.SilkS")
 			(effects
 				(font
@@
 		(property "Value" "Up Button"
 			(at -3 -1.5 0)
-			(layer "B.Fab")
+			(layer "B.SilkS")
 			(effects
 				(font
@@
 		)
 		(property "Value" "100nF"
-			(at -2.002294 1.497842 0)
-			(layer "B.Fab")
+			(at -2.002294 -0.497842 0)
+			(layer "B.SilkS")
 			(effects
 				(font
@@
 	(footprint "Capacitor_THT:C_Disc_D3.0mm_W1.6mm_P2.50mm"
 		(layer "B.Cu")
-		(at 87.997842 118.997706 90)
+		(at 112.5 119 90)
 		(descr "C, Disc series, Radial, pin pitch=2.50mm, diameter*width=3.0*1.6mm^2, Capacitor, http://www.vishay.com/docs/45233/krseries.pdf")
 		(tags "C Disc series Radial pin pitch 2.50mm diameter 3.0mm width 1.6mm Capacitor")
@@
 		)
 		(property "Value" "100nF"
-			(at -4.002294 0.497842 90)
-			(layer "B.Fab")
+			(at 5 1 180)
+			(layer "B.SilkS")
 			(effects
 				(font
@@
 		)
 		(property "Value" "74HC595"
-			(at -1.997706 -16.497842 0)
-			(layer "B.Fab")
+			(at 10 -16 0)
+			(layer "B.SilkS")
 			(effects
 				(font
@@
 		(property "Value" "UDN2981A"
 			(at -10 5.232 0)
-			(layer "B.Fab")
+			(layer "B.SilkS")
 			(effects
 				(font
@@
 	)
 	(gr_rect
-		(start 65.5 71.5)
-		(end 285.5 150)
+		(start 63.5 71.75)
+		(end 287.5 150.25)
 		(stroke
 			(width 0.05)
@@
 	)
 	(gr_text "IV-11 VFD Tube Clock\nMade in Wisconsin\nAron Szucs 2026\n"
-		(at 274.5 79 270)
+		(at 276.5 81 270)
 		(layer "F.SilkS")
 		(effects
